File: robo-plater/elec/layout/default/robo-plater.kicad_pcb (KiCad board)
At the start: 4 copper layers, 132.7 x 100 mm, 241 parts, among them J1 ?, J2 ?, J3 ?, J4 ?, J5 ?, J6 ?, J7 ?, J8 ?, U1 ?, U10 ?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

Commit message: CI workflows for robo-plater
Other:
- board text added: "Matt Wildoer"
- board text added: "{{GITHASH}}"
